File: hardware/psm-v1/psm-v1.kicad_pcb (KiCad board)
At the start: 2 copper layers, 101.6 x 101.6 mm, 68 parts, among them J1 Tiva_IF, U1 VCNL4020, U10 VCNL4020, U11 VCNL4020, U12 VCNL4020, U13 VCNL4020, U14 VCNL4020, U15 VCNL4020, U16 VCNL4020, U17 PCA9548A, U18 PCA9548A, U2 VCNL4020, U3 VCNL4020, U4 VCNL4020, U5 VCNL4020, U6 VCNL4020, U7 VCNL4020, U8 VCNL4020, U9 VCNL4020

Commit message: Add full V1 and V3 KiCad schematics and netlist checks
Connections:
- J1 pad 7: 5V -> (no net)
Changed lines of the file:
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@@
 			(layers "*.Cu" "*.Mask")
 			(remove_unused_layers no)
-			(net "5V")
 		)
 		(pad "8" thru_hole circle
