File: hardware/psm-v1/psm-v1.kicad_sch (KiCad schematic)
At the start: 41 parts, among them J1 HOST_IF, U1 VCNL4020, U10 VCNL4020, U11 VCNL4020, U12 VCNL4020, U13 VCNL4020, U14 VCNL4020, U15 VCNL4020, U16 VCNL4020, U17 PCA9548A 0x70, U18 PCA9548A 0x71, U2 VCNL4020, U3 VCNL4020, U4 VCNL4020, U5 VCNL4020, U6 VCNL4020, U7 VCNL4020, U8 VCNL4020, U9 VCNL4020

Commit message: Add full V1 and V3 KiCad schematics and netlist checks
Parts:
- added C1, C10, C11, C12, C13, C14, C15, C16, C2, C3, C4, C5, C6, C7, C8, C9: 100n, psm:C_0603_1608Metric, symbol PSM:C
Connections:
- net 3V3: now also C1.1, C10.1, C11.1, C12.1, C13.1, C14.1, C15.1, C16.1, C2.1, C3.1, C4.1, C5.1, C6.1, C7.1, C8.1, C9.1
- net GND: now also C1.2, C10.2, C11.2, C12.2, C13.2, C14.2, C15.2, C16.2, C2.2, C3.2, C4.2, C5.2, C6.2, C7.2, C8.2, C9.2; no longer U17.25 (EP), U18.25 (EP)
Other:
- note added: "Per sensor: 100nF local decoupling (C1-C16), 10R IR-anode series resistor (R1-R16). 22uF bulk C17/C18."
- note removed: "Per sensor: 100nF local decoupling, 10R IR-anode series resistor. 22uF bulk per mux/header."
