File: hardware/psm-v3/hub/psm-v3-hub.kicad_pcb (KiCad board)
At the start: 2 copper layers, 60 x 40 mm, 28 parts, among them J1 HOST_IF, J2 TILE_0, J3 TILE_1, J4 TILE_2, J5 TILE_3, U1 PCA9548A, U2 USBLC6-2SC6

Commit message: Add full V1 and V3 KiCad schematics and netlist checks
Connections:
- J1 pad 7: 5V -> (no net)
Changed lines of the file:
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@@
 			(layers "*.Cu" "*.Mask")
 			(remove_unused_layers no)
-			(net "5V")
 		)
 		(pad "8" thru_hole circle
