File: hardware/psm-v3/tile/psm-v3-tile.kicad_pcb (KiCad board)
At the start: 2 copper layers, 30 x 30 mm, 21 parts, among them J1 TILE_IF, U1 VCNL4030X01 0x60, U2 VCNL4030X01 0x51, U3 VCNL4030X01 0x40, U4 VCNL4030X01 0x41

Commit message: Add full V1 and V3 KiCad schematics and netlist checks
Connections:
- J1 pad 6: NC -> (no net)
Changed lines of the file:
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@@
 			(layers "*.Cu" "*.Mask")
 			(remove_unused_layers no)
-			(net "NC")
 		)
 		(embedded_fonts no)
